Commit message: run

File: urdf/fishbot/base.urdf.xacro (robot description, xacro)
@@ -11,4 +11,7 @@
     <xacro:property name="wheel_offset_x" value="0.2" />
     <xacro:property name="wheel_offset_y" value="0.23" />
+    <!-- 万向轮属性 -->
+    <xacro:property name="caster_radius" value="0.04" />
+    <xacro:property name="caster_mass" value="0.5" />
     <!-- 材料定义 Materials -->
     <material name="chassis_material">
@@ -37,7 +40,6 @@
         </inertial>
     </xacro:macro>
-    <!-- 虚拟的base_footprint链接 - 位于地面上 -->
+    <!-- 虚拟的base_footprint链接 -->
     <link name="base_footprint">
-        <!-- 这是一个虚拟链接，没有视觉或碰撞属性 -->
     </link>
     <!-- 机器人底盘 Base Link -->
@@ -67,6 +69,6 @@
         <origin xyz="0 0 ${wheel_radius + chassis_height/2}" rpy="0 0 0"/>
     </joint>
-    <!-- 车轮宏定义 Wheel Macro -->
-    <xacro:macro name="wheel" params="prefix x_pos y_pos">
+    <!-- 后轮宏定义（驱动轮） -->
+    <xacro:macro name="rear_wheel" params="prefix x_pos y_pos">
         <link name="${prefix}_wheel">
             <visual>
@@ -98,8 +100,59 @@
         </joint>
     </xacro:macro>
-    <!-- 使用宏创建四个车轮 Instantiate four wheels using macro -->
-    <xacro:wheel prefix="front_left"  x_pos="${wheel_offset_x}"  y_pos="${wheel_offset_y}"/>
-    <xacro:wheel prefix="front_right" x_pos="${wheel_offset_x}"  y_pos="${-wheel_offset_y}"/>
-    <xacro:wheel prefix="rear_left"   x_pos="${-wheel_offset_x}" y_pos="${wheel_offset_y}"/>
-    <xacro:wheel prefix="rear_right"  x_pos="${-wheel_offset_x}" y_pos="${-wheel_offset_y}"/>
+    <!-- 万向轮宏定义（前轮） -->
+    <xacro:macro name="caster_wheel" params="prefix x_pos y_pos">
+        <!-- 使用球形万向轮 -->
+        <link name="${prefix}_caster_wheel">
+            <visual>
+                <origin xyz="0 0 0" rpy="0 0 0"/>
+                <geometry>
+                    <sphere radius="${caster_radius}"/>
+                </geometry>
+                <material name="wheel_material"/>
+            </visual>
+            <collision>
+                <origin xyz="0 0 0" rpy="0 0 0"/>
+                <geometry>
+                    <sphere radius="${caster_radius}"/>
+                </geometry>
+                <surface>
+                    <friction>
+                        <ode>
+                            <mu>0.01</mu>
+                            <mu2>0.01</mu2>
+                        </ode>
+                    </friction>
+                </surface>
+            </collision>
+            <inertial>
+                <origin xyz="0 0 0" rpy="0 0 0"/>
+                <mass value="${caster_mass}"/>
+                <inertia ixx="${2*caster_mass*caster_radius*caster_radius/5}" ixy="0" ixz="0"
+                         iyy="${2*caster_mass*caster_radius*caster_radius/5}" iyz="0"
+                         izz="${2*caster_mass*caster_radius*caster_radius/5}"/>
+            </inertial>
+        </link>
+        <joint name="${prefix}_caster_joint" type="fixed">
+            <parent link="base_link"/>
+            <child link="${prefix}_caster_wheel"/>
+            <!-- 调整高度以匹配后轮接触地面 -->
+            <origin xyz="${x_pos} ${y_pos} ${-chassis_height/2 - wheel_radius + caster_radius}" rpy="0 0 0"/>
+        </joint>
+        <!-- Gazebo配置 -->
+        <gazebo reference="${prefix}_caster_wheel">
+            <material>Gazebo/Black</material>
+            <mu1>0.01</mu1>
+            <mu2>0.01</mu2>
+            <kp>1000000.0</kp>
+            <kd>100.0</kd>
+            <minDepth>0.001</minDepth>
+            <maxVel>1.0</maxVel>
+        </gazebo>
+    </xacro:macro>
+    <!-- 创建两个后轮（驱动轮） -->
+    <xacro:rear_wheel prefix="rear_left" x_pos="${-wheel_offset_x}" y_pos="${wheel_offset_y}"/>
+    <xacro:rear_wheel prefix="rear_right" x_pos="${-wheel_offset_x}" y_pos="${-wheel_offset_y}"/>
+    <!-- 创建两个前轮（万向轮） -->
+    <xacro:caster_wheel prefix="front_left" x_pos="${wheel_offset_x}" y_pos="${wheel_offset_y}"/>
+    <xacro:caster_wheel prefix="front_right" x_pos="${wheel_offset_x}" y_pos="${-wheel_offset_y}"/>
 </robot>
